File: KiCad/tag.kicad_pcb (KiCad board)
At the start: 2 copper layers, 35 x 62 mm, 18 parts, among them SW1 PTS526 SM15 SMTR2 LFS, U1 ATtiny85V-10S, U2 ST25DV04KC-IE6S3, U3 APTF1616LSEEZGKQBKC

Commit message: Add files via upload
Routing:
- net GND: track 88.8 -> 73.8 mm
- added copper zone on B.Cu, net GND
- added copper zone on F.Cu, net GND
Changed lines of the file:
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@@
 		(capping no)
 		(filling no)
-		(zone_defaults)
 		(pcbplotparams
 			(layerselection 0x00000000_00000000_55555555_5755f5ff)
@@
 	)
 	(segment
-		(start 98.42 64.46)
-		(end 99.8083 65.8483)
-		(width 0.2)
-		(layer "B.Cu")
-		(net "GND")
-	)
-	(segment
 		(start 119.2108 72.1104)
 		(end 119.2108 71.3806)
@@
 	)
 	(segment
-		(start 102.23 66.5994)
-		(end 102.23 67.878)
-		(width 0.2)
-		(layer "B.Cu")
-		(net "GND")
-	)
-	(segment
 		(start 110.6309 69.5781)
 		(end 112.4334 71.3806)
@@
 	)
 	(segment
-		(start 102.23 67.878)
-		(end 103.9301 69.5781)
-		(width 0.2)
-		(layer "B.Cu")
-		(net "GND")
-	)
-	(segment
-		(start 101.4789 65.8483)
-		(end 102.23 66.5994)
-		(width 0.2)
-		(layer "B.Cu")
-		(net "GND")
-	)
-	(segment
-		(start 99.8083 65.8483)
-		(end 101.4789 65.8483)
-		(width 0.2)
-		(layer "B.Cu")
-		(net "GND")
-	)
-	(segment
-		(start 103.9301 69.5781)
-		(end 110.6309 69.5781)
-		(width 0.2)
-		(layer "B.Cu")
-		(net "GND")
-	)
-	(segment
 		(start 106.9316 90.5129)
 		(end 105.7208 89.3021)
@@
 		(net "Net-(U2-AC1)")
 	)
+	(zone
+		(layers "F.Cu" "B.Cu")
+		(hatch edge 0.5)
+		(connect_pads
+			(clearance 0)
+		)
+		(min_thickness 0.25)
+		(keepout
+			(tracks allowed)
+			(vias allowed)
+			(pads allowed)
+			(copperpour not_allowed)
+			(footprints allowed)
+		)
+		(placement
+			(enabled no)
+			(sheetname "")
+		)
+		(fill
+			(thermal_gap 0.5)
+			(thermal_bridge_width 0.5)
+			(island_removal_mode 0)
+		)
+		(polygon
+			(pts
+				(xy 99.55 65.025) (xy 98.925 65.65) (xy 99.7 66.5) (xy 100.6 65.75) (xy 99.75 64.975)
+			)
+		)
+	)
+	(zone
+		(net "GND")
+		(layers "F.Cu" "B.Cu")
+		(name "Ground")
+		(hatch edge 0.5)
+		(connect_pads
+			(clearance 0.5)
+		)
+		(min_thickness 0.25)
+		(fill yes
+			(thermal_gap 0.5)
+			(thermal_bridge_width 0.5)
+			(island_removal_mode 0)
+		)
+		(polygon
+			(pts
+				(xy 129.025 61.2) (xy 129 92.46) (xy 94.025 92.46) (xy 94.025 61.2)
+			)
+		)
+	)
 	(embedded_fonts no)
